File: pcb/teensy-dsp/teensy-dsp.kicad_sch (KiCad schematic)
At the start: 5 parts, among them J1 ACJS-IH, J2 ACJS-IH, J3 ACJS-IH, J4 ACJS-IH, U1 Teensy4.1

Commit message: updated solidworks and kicad files
Parts:
- removed J1, J2, J3, J4: ACJS-IH, ACJS-IH_AMP, symbol 2023-11-11_03-32-11:ACJS-IH
- added U2: Teensy4.0_AudioShield_REVD, symbol Teensy MCUs:Teensy4.0_AudioShield_REVD
Connections:
- net +3.3V: now reaches U1.46 (3V3)
- net +3.3V: now also U2.28 (3V)
- net GND: now reaches U1.47 (GND)
- net GND: now also U2.29 (GND)
- net +5V: now reaches U1.48 (VIN)
- new net Audio IO/Line In L: U2.35 (LINE_IN_L)
- new net Audio IO/Line In LGND: U2.37 (LINE_IN_L_GND)
- new net Audio IO/Line In R: U2.34 (LINE_IN_R)
- new net Audio IO/Line In RGND: U2.36 (LINE_IN_R_GND)
- new net Audio IO/Line Out GND: U2.32 (LINE_OUT_GND)
- new net Audio IO/Line Out L: U2.31 (LINE_OUT_L)
- new net Audio IO/Line Out R: U2.33 (LINE_OUT_R)
- no-connect marks 0 -> 10
Other:
- added sheet Audio IO (io.kicad_sch)
- added sheet Power (power.kicad_sch)
- note removed: "Inputs"
- note removed: "Left Input"
- note removed: "Left Output"
- note removed: "Outputs"
- note removed: "Right Input"
- note removed: "Right Output"
- moved on the sheet: U1

Commit message: update renders
Parts:
- added J1: FSW1, Connector_Molex:Molex_Micro-Fit_3.0_43650-0200_1x02_P3.00mm_Horizontal, symbol Connector:Conn_01x02_Pin
- added J2: FSW2, Connector_Molex:Molex_Micro-Fit_3.0_43650-0200_1x02_P3.00mm_Horizontal, symbol Connector:Conn_01x02_Pin
Connections:
- net GND: now also J1.2 (Pin_2), J2.2 (Pin_2)
- new net FSW_1: J1.1 (Pin_1)
- new net FSW_2: J2.1 (Pin_1)
Changed lines of the file:
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@@
   (no_connect (at 222.25 77.47))
   (no_connect (at 166.37 102.87))
+  (wire (pts (xy 128.27 175.26) (xy 132.08 175.26))
+    (stroke (width 0) (type default))
+  )
   (wire (pts (xy 222.25 102.87) (xy 246.38 102.87))
     (stroke (width 0) (type default))
@@
     (stroke (width 0) (type default))
   )
+  (wire (pts (xy 128.27 153.67) (xy 138.43 153.67))
+    (stroke (width 0) (type default))
+  )
   (wire (pts (xy 222.25 127) (xy 237.49 127))
     (stroke (width 0) (type default))
@@
     (stroke (width 0) (type default))
   )
+  (wire (pts (xy 128.27 172.72) (xy 138.43 172.72))
+    (stroke (width 0) (type default))
+  )
+  (wire (pts (xy 132.08 175.26) (xy 132.08 177.8))
+    (stroke (width 0) (type default))
+  )
   (wire (pts (xy 222.25 107.95) (xy 246.38 107.95))
     (stroke (width 0) (type default))
   )
+  (wire (pts (xy 132.08 156.21) (xy 132.08 158.75))
+    (stroke (width 0) (type default))
+  )
+  (wire (pts (xy 128.27 156.21) (xy 132.08 156.21))
+    (stroke (width 0) (type default))
+  )
   (wire (pts (xy 123.19 63.5) (xy 125.73 63.5))
     (stroke (width 0) (type default))
@@
   (wire (pts (xy 123.19 60.96) (xy 123.19 63.5))
     (stroke (width 0) (type default))
+  )
+  (global_label "FSW_1" (shape input) (at 138.43 153.67 0) (fields_autoplaced)
+    (effects (font (size 1.27 1.27)) (justify left))
+    (property "Intersheetrefs" "${INTERSHEET_REFS}" (at 147.2624 153.67 0)
+      (effects (font (size 1.27 1.27)) (justify left) hide)
+    )
+  )
+  (global_label "FSW_2" (shape input) (at 138.43 172.72 0) (fields_autoplaced)
+    (effects (font (size 1.27 1.27)) (justify left))
+    (property "Intersheetrefs" "${INTERSHEET_REFS}" (at 147.2624 172.72 0)
+      (effects (font (size 1.27 1.27)) (justify left) hide)
+    )
   )
   (symbol (lib_id "Teensy MCUs:Teensy4.0_AudioShield_REVD") (at 194.31 97.79 0) (unit 1)
@@
     )
   )
+  (symbol (lib_id "Connector:Conn_01x02_Pin") (at 123.19 172.72 0) (unit 1)
+    (in_bom yes) (on_board yes) (dnp no) (fields_autoplaced)
+    (property "Reference" "J2" (at 123.825 168.91 0)
+      (effects (font (size 1.27 1.27)))
+    )
+    (property "Value" "FSW2" (at 123.825 171.45 0)
+      (effects (font (size 1.27 1.27)))
+    )
+    (property "Footprint" "Connector_Molex:Molex_Micro-Fit_3.0_43650-0200_1x02_P3.00mm_Horizontal" (at 123.19 172.72 0)
+      (effects (font (size 1.27 1.27)) hide)
+    )
+    (property "Datasheet" "~" (at 123.19 172.72 0)
+      (effects (font (size 1.27 1.27)) hide)
+    )
+    (pin "1")
+    (pin "2")
+    (instances
+      (project "teensy-dsp-frontend"
+        (path "/8dbf74d9-99dc-4819-8a81-8d7bc3c2d99c"
+          (reference "J2") (unit 1)
+        )
+      )
+      (project "teensy-dsp"
+        (path "/b4828465-e4d8-4e3f-b668-f3defd59a393"
+          (reference "J4") (unit 1)
+        )
+      )
+    )
+  )
   (symbol (lib_id "power:+5V") (at 105.41 55.88 0) (unit 1)
     (in_bom yes) (on_board yes) (dnp no) (fields_autoplaced)
@@
         (path "/b4828465-e4d8-4e3f-b668-f3defd59a393"
           (reference "#PWR01") (unit 1)
+        )
+      )
+    )
+  )
+  (symbol (lib_id "power:GND") (at 132.08 158.75 0) (unit 1)
+    (in_bom yes) (on_board yes) (dnp no) (fields_autoplaced)
+    (property "Reference" "#PWR020" (at 132.08 165.1 0)
+      (effects (font (size 1.27 1.27)) hide)
+    )
+    (property "Value" "GND" (at 132.08 163.83 0)
+      (effects (font (size 1.27 1.27)))
+    )
+    (property "Footprint" "" (at 132.08 158.75 0)
+      (effects (font (size 1.27 1.27)) hide)
+    )
+    (property "Datasheet" "" (at 132.08 158.75 0)
+      (effects (font (size 1.27 1.27)) hide)
+    )
+    (pin "1")
+    (instances
+      (project "teensy-dsp-frontend"
+        (path "/8dbf74d9-99dc-4819-8a81-8d7bc3c2d99c"
+          (reference "#PWR020") (unit 1)
+        )
+      )
+      (project "teensy-dsp"
+        (path "/b4828465-e4d8-4e3f-b668-f3defd59a393"
+          (reference "#PWR04") (unit 1)
+        )
+      )
+    )
+  )
+  (symbol (lib_id "power:GND") (at 132.08 177.8 0) (unit 1)
+    (in_bom yes) (on_board yes) (dnp no) (fields_autoplaced)
+    (property "Reference" "#PWR021" (at 132.08 184.15 0)
+      (effects (font (size 1.27 1.27)) hide)
+    )
+    (property "Value" "GND" (at 132.08 182.88 0)
+      (effects (font (size 1.27 1.27)))
+    )
+    (property "Footprint" "" (at 132.08 177.8 0)
+      (effects (font (size 1.27 1.27)) hide)
+    )
+    (property "Datasheet" "" (at 132.08 177.8 0)
+      (effects (font (size 1.27 1.27)) hide)
+    )
+    (pin "1")
+    (instances
+      (project "teensy-dsp-frontend"
+        (path "/8dbf74d9-99dc-4819-8a81-8d7bc3c2d99c"
+          (reference "#PWR021") (unit 1)
+        )
+      )
+      (project "teensy-dsp"
+        (path "/b4828465-e4d8-4e3f-b668-f3defd59a393"
+          (reference "#PWR07") (unit 1)
         )
       )
@@
         )
       )
+    )
+  )
+  (symbol (lib_id "Connector:Conn_01x02_Pin") (at 123.19 153.67 0) (unit 1)
+    (in_bom yes) (on_board yes) (dnp no) (fields_autoplaced)
+    (property "Reference" "J1" (at 123.825 149.86 0)
+      (effects (font (size 1.27 1.27)))
+    )
+    (property "Value" "FSW1" (at 123.825 152.4 0)
+      (effects (font (size 1.27 1.27)))
+    )
+    (property "Footprint" "Connector_Molex:Molex_Micro-Fit_3.0_43650-0200_1x02_P3.00mm_Horizontal" (at 123.19 153.67 0)
+      (effects (font (size 1.27 1.27)) hide)
+    )
+    (property "Datasheet" "~" (at 123.19 153.67 0)
+      (effects (font (size 1.27 1.27)) hide)
+    )
+    (pin "1")
+    (pin "2")
+    (instances
+      (project "teensy-dsp-frontend"
+        (path "/8dbf74d9-99dc-4819-8a81-8d7bc3c2d99c"
+          (reference "J1") (unit 1)
+        )
+      )
+      (project "teensy-dsp"
+        (path "/b4828465-e4d8-4e3f-b668-f3defd59a393"
+          (reference "J3") (unit 1)
+        )
+      )

Commit message: update pcb layout
Parts:
- added J1: Conn_02x15_Odd_Even, Connector_IDC:IDC-Header_2x15_P2.54mm_Vertical, symbol Connector_Generic:Conn_02x15_Odd_Even
- added J9: USB_B_Mini, Connector_USB:USB_Mini-B_Wuerth_65100516121_Horizontal, symbol Connector:USB_B_Mini
- U1: footprint (none) -> Imported Footprints:MODULE_DEV-16771; symbol teensy:Teensy4.1 -> DEV-16771:DEV-16771; MANUFACTURER (none) -> SparkFun Electronics; MAXIMUM_PACKAGE_HEIGHT (none) -> 4.07mm; PARTREV (none) -> 4.1; STANDARD (none) -> Manufacturer recommendations
- U2: footprint (none) -> Imported Footprints:4.0audioshield
Connections:
- net Audio IO/Line In LGND is gone; now on net GND: U2.37 (LINE_IN_L_GND)
- net Audio IO/Line In RGND is gone; now on net GND: U2.36 (LINE_IN_R_GND)
- net Audio IO/Line Out GND is gone; now on net GND: U2.32 (LINE_OUT_GND)
- net +3.3V: now also U1.3.3V_1 (3.3V), U1.3.3V_2 (3.3V__1), U1.3.3V_3 (3.3V__2), J1.7 (Pin_7); no longer U1.46 (3V3)
- net +5V: now also U1.VIN, J1.5 (Pin_5); no longer U1.48 (VIN)
- net FSW_1: now also U1.28 (RX7)
- net FSW_2: now also U1.29 (TX7)
- net GND: now also U1.GND1 (GND), U1.GND2 (GND__1), U1.GND3 (GND__2), U1.GND4 (GND__3), U1.GND5 (GND__4), U1.USB_GND1 (USB_GND), U1.USB_GND2 (USB_GND__1), U2.1 (GND), J1.10 (Pin_10), J1.12 (Pin_12), J1.14 (Pin_14), J1.16 (Pin_16), J1.18 (Pin_18), J1.2 (Pin_2), J1.20 (Pin_20), J1.22 (Pin_22), J1.24 (Pin_24), J1.26 (Pin_26), J1.28 (Pin_28), J1.30 (Pin_30), J1.4 (Pin_4), J1.6 (Pin_6), J1.8 (Pin_8), J9.5 (GND); no longer U1.47 (GND)
- net Audio DOUT: now reaches U2.10 (8_TX2_IN1)
- net Audio DOUT: now also U1.8 (TX2)
- net Audio SDCS: now reaches U2.12 (10_CS_MQSR)
- net Audio SDCS: now also U1.10 (CS1)
- net Audio MOSI: now reaches U2.13 (11_MOSI_CTX1)
- net Audio MOSI: now also U1.11 (MOSI)
- net Audio MISO: now reaches U2.14 (12_MISO_MQSL)
- net Audio MISO: now also U1.12 (MISO)
- net Audio SCK: now reaches U2.17 (13_SCK_CRX1_LED)
- net Audio SCK: now also U1.13 (SCK)
- net Audio SDA: now reaches U2.22 (18_A4_SDA0)
- net Audio SDA: now also U1.18 (A4)
- net Audio SCL: now reaches U2.23 (19_A5_SCL0)
- net Audio SCL: now also U1.19 (A5)
- net Audio LRCLK: now reaches U2.24 (20_A6_TX5_LRCLK1)
- net Audio LRCLK: now also U1.20 (A6)
- net Audio BCLK: now reaches U2.25 (21_A7_RX5_BCLK1)
- net Audio BCLK: now also U1.21 (A7)
- net Audio MCLK: now reaches U2.27 (23_A9_CRX1_MCLK1)
- net Audio MCLK: now also U1.23 (A9)
- net Audio MEMCS: now reaches U2.8 (6_OUT1D)
- net Audio MEMCS: now also U1.6 (OUT1D)
- net Audio DIN: now reaches U2.9 (7_RX2_OUT1A)
- net Audio DIN: now also U1.7 (RX2)
- net LED_BLANK: now reaches U1.2 (OUT2)
- net LED_BLANK: now also J1.11 (Pin_11)
- net POT_4: now reaches U1.24 (A10)
- net POT_4: now also J1.25 (Pin_25)
- net POT_3: now reaches U1.25 (A11)
- net POT_3: now also J1.23 (Pin_23)
- net POT_2: now reaches U1.26 (A12)
- net POT_2: now also J1.21 (Pin_21)
- net POT_1: now reaches U1.27 (A13)
- net POT_1: now also J1.19 (Pin_19)
- net LED_XLAT: now reaches U1.3 (LRCLK2)
- net LED_XLAT: now also J1.13 (Pin_13)
- net POT_5: now reaches U1.38 (A14)
- net POT_5: now also J1.27 (Pin_27)
- net POT_6: now reaches U1.39 (A15)
- net POT_6: now also J1.29 (Pin_29)
- net LED_SCLK: now reaches U1.4 (BCLK2)
- net LED_SCLK: now also J1.15 (Pin_15)
- net LED_GSCLK: now reaches U1.5 (IN2)
- net LED_GSCLK: now also J1.9 (Pin_9)
- net LED_SIN: now reaches U1.9 (OUT1C)
- net LED_SIN: now also J1.17 (Pin_17)
- net Audio IO/Line In L renamed L Line In
- net Audio IO/Line In R renamed R Line In
- net Audio IO/Line Out L renamed L Line Out
- net Audio IO/Line Out R renamed R Line Out
- new net: J9.2 (D-), U1.D-
- new net: J9.3 (D+), U1.D+
- new net +9V: J1.1 (Pin_1), J1.3 (Pin_3)
- no-connect marks 10 -> 51
Other:
- sheet Audio IO ports: added none; removed Line In L, Line In LGND, Line In R, Line In RGND, Line Out GND, Line Out L, Line Out R
- moved on the sheet: J1, J2, U2

Commit message: update pcb layout
Connections:
- net Earth: now reaches J9.6 (Shield)
- no-connect marks 51 -> 50
Changed lines of the file:
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@@
   (no_connect (at 182.88 83.82))
   (no_connect (at 90.17 50.8))
+  (no_connect (at 123.19 50.8))
   (no_connect (at 90.17 78.74))
   (no_connect (at 238.76 35.56))
@@
   (no_connect (at 238.76 38.1))
   (no_connect (at 238.76 101.6))
-  (no_connect (at 90.17 33.02))
   (no_connect (at 182.88 40.64))
   (no_connect (at 49.53 68.58))
-  (no_connect (at 133.35 66.04))
-  (no_connect (at 123.19 50.8))
   (no_connect (at 49.53 111.76))
   (no_connect (at 182.88 43.18))
   (no_connect (at 49.53 45.72))
   (no_connect (at 90.17 40.64))
+  (no_connect (at 90.17 33.02))
   (no_connect (at 238.76 91.44))
   (no_connect (at 182.88 38.1))
@@
     (stroke (width 0) (type default))
   )
+  (wire (pts (xy 133.35 66.04) (xy 137.16 66.04))
+    (stroke (width 0) (type default))
+  )
   (wire (pts (xy 90.17 137.16) (xy 93.98 137.16))
     (stroke (width 0) (type default))
@@
   )
   (wire (pts (xy 238.76 55.88) (xy 241.3 55.88))
+    (stroke (width 0) (type default))
+  )
+  (wire (pts (xy 137.16 66.04) (xy 137.16 68.58))
     (stroke (width 0) (type default))
   )
@@
         )
       )
+    )
+  )
+  (symbol (lib_id "power:Earth") (at 137.16 68.58 0) (unit 1)
+    (in_bom yes) (on_board yes) (dnp no) (fields_autoplaced)
+    (property "Reference" "#PWR025" (at 137.16 74.93 0)
+      (effects (font (size 1.27 1.27)) hide)
+    )
+    (property "Value" "Earth" (at 137.16 72.39 0)
+      (effects (font (size 1.27 1.27)) hide)
+    )
+    (property "Footprint" "" (at 137.16 68.58 0)
+      (effects (font (size 1.27 1.27)) hide)
+    )
+    (property "Datasheet" "~" (at 137.16 68.58 0)
+      (effects (font (size 1.27 1.27)) hide)
+    )
+    (pin "1")
+    (instances
+      (project "teensy-dsp"
+        (path "/b4828465-e4d8-4e3f-b668-f3defd59a393"
+          (reference "#PWR025") (unit 1)
+        )
+      )

Commit message: pcb and case updates
Parts:
- removed J1: FSW1, Connector_Molex:Molex_Micro-Fit_3.0_43650-0200_1x02_P3.00mm_Horizontal, symbol Connector:Conn_01x02_Pin
- removed J2: FSW2, Connector_Molex:Molex_Micro-Fit_3.0_43650-0200_1x02_P3.00mm_Horizontal, symbol Connector:Conn_01x02_Pin
Connections:
- net +3.3V: now also J1.3 (Pin_3); no longer J1.7 (Pin_7)
- net +5V: no longer J1.5 (Pin_5)
- net +9V: no longer J1.3 (Pin_3)
- net FSW_1: now also J1.7 (Pin_7)
- net FSW_2: now also J1.5 (Pin_5)
- net LED_BLANK: now also J1.15 (Pin_15); no longer J1.11 (Pin_11)
- net LED_SCLK: now also J1.11 (Pin_11); no longer J1.15 (Pin_15)
