File: pcb/teensy-dsp/io.kicad_sch (KiCad schematic)
At the start: 4 parts, among them J1 ACJS-IH, J2 ACJS-IH

Commit message: update pcb layout
Connections:
- net Line In RGND is gone; now on net GND: J2.R
- net Line Out GND is gone; now on net GND: J1.R, J2.R
- net Line In L renamed R Line Out
- net Line In LGND renamed GND
- net Line In R renamed L Line Out
- net Line Out L renamed R Line In
- net Line Out R renamed L Line In
Changed lines of the file:
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@@
 (kicad_sch (version 20230121) (generator eeschema)
   (paper "A4")
-  (junction (at 109.22 115.57) (diameter 0) (color 0 0 0 0)
-  )
   (no_connect (at 81.28 118.11))
   (no_connect (at 81.28 77.47))
@@
   (no_connect (at 81.28 49.53))
   (no_connect (at 81.28 153.67))
-  (wire (pts (xy 81.28 115.57) (xy 109.22 115.57))
+  (wire (pts (xy 81.28 64.77) (xy 86.36 64.77))
     (stroke (width 0) (type default))
   )
@@
     (stroke (width 0) (type default))
   )
-  (wire (pts (xy 109.22 115.57) (xy 116.84 115.57))
-    (stroke (width 0) (type default))
-  )
-  (wire (pts (xy 109.22 140.97) (xy 109.22 115.57))
-    (stroke (width 0) (type default))
-  )
-  (wire (pts (xy 81.28 39.37) (xy 90.17 39.37))
+  (wire (pts (xy 81.28 140.97) (xy 86.36 140.97))
+    (stroke (width 0) (type default))
+  )
+  (wire (pts (xy 86.36 115.57) (xy 86.36 116.84))
+    (stroke (width 0) (type default))
+  )
+  (wire (pts (xy 81.28 39.37) (xy 86.36 39.37))
     (stroke (width 0) (type default))
   )
@@
     (stroke (width 0) (type default))
   )
-  (wire (pts (xy 81.28 64.77) (xy 90.17 64.77))
+  (wire (pts (xy 86.36 64.77) (xy 86.36 66.04))
+    (stroke (width 0) (type default))
+  )
+  (wire (pts (xy 86.36 39.37) (xy 86.36 40.64))
+    (stroke (width 0) (type default))
+  )
+  (wire (pts (xy 86.36 140.97) (xy 86.36 142.24))
     (stroke (width 0) (type default))
   )
@@
     (stroke (width 0) (type default))
   )
-  (wire (pts (xy 81.28 140.97) (xy 109.22 140.97))
+  (wire (pts (xy 81.28 115.57) (xy 86.36 115.57))
     (stroke (width 0) (type default))
   )
@@
     (stroke (width 0) (type default))
   )
-  (text "Left Output" (at 60.96 132.08 0)
-    (effects (font (size 1.27 1.27)) (justify left bottom))
-  )
-  (text "Right Ouptut" (at 60.96 157.48 0)
-    (effects (font (size 1.27 1.27)) (justify left bottom))
-  )
-  (text "Left Input" (at 60.96 55.88 0)
-    (effects (font (size 1.27 1.27)) (justify left bottom))
-  )
-  (text "Right Input" (at 60.96 81.28 0)
-    (effects (font (size 1.27 1.27)) (justify left bottom))
-  )
-  (hierarchical_label "Line Out L" (shape input) (at 90.17 123.19 0) (fields_autoplaced)
-    (effects (font (size 1.27 1.27)) (justify left))
-  )
-  (hierarchical_label "Line In R" (shape output) (at 90.17 72.39 0) (fields_autoplaced)
-    (effects (font (size 1.27 1.27)) (justify left))
-  )
-  (hierarchical_label "Line Out R" (shape input) (at 90.17 148.59 0) (fields_autoplaced)
-    (effects (font (size 1.27 1.27)) (justify left))
-  )
-  (hierarchical_label "Line Out GND" (shape input) (at 116.84 115.57 0) (fields_autoplaced)
-    (effects (font (size 1.27 1.27)) (justify left))
-  )
-  (hierarchical_label "Line In LGND" (shape output) (at 90.17 39.37 0) (fields_autoplaced)
-    (effects (font (size 1.27 1.27)) (justify left))
-  )
-  (hierarchical_label "Line In L" (shape output) (at 90.17 46.99 0) (fields_autoplaced)
-    (effects (font (size 1.27 1.27)) (justify left))
-  )
-  (hierarchical_label "Line In RGND" (shape output) (at 90.17 64.77 0) (fields_autoplaced)
-    (effects (font (size 1.27 1.27)) (justify left))
+  (text "Left Output" (at 60.96 81.28 0)
+    (effects (font (size 1.27 1.27)) (justify left bottom))
+  )
+  (text "Right Ouptut" (at 60.96 55.88 0)
+    (effects (font (size 1.27 1.27)) (justify left bottom))
+  )
+  (text "Left Input" (at 60.96 157.48 0)
+    (effects (font (size 1.27 1.27)) (justify left bottom))
+  )
+  (text "Right Input" (at 60.96 132.08 0)
+    (effects (font (size 1.27 1.27)) (justify left bottom))
+  )
+  (global_label "R Line Out" (shape input) (at 90.17 46.99 0) (fields_autoplaced)
+    (effects (font (size 1.27 1.27)) (justify left))
+    (property "Intersheetrefs" "${INTERSHEET_REFS}" (at 102.9455 46.99 0)
+      (effects (font (size 1.27 1.27)) (justify left) hide)
+    )
+  )
+  (global_label "R Line In" (shape input) (at 90.17 123.19 0) (fields_autoplaced)
+    (effects (font (size 1.27 1.27)) (justify left))
+    (property "Intersheetrefs" "${INTERSHEET_REFS}" (at 101.4941 123.19 0)
+      (effects (font (size 1.27 1.27)) (justify left) hide)
+    )
+  )
+  (global_label "L Line Out" (shape input) (at 90.17 72.39 0) (fields_autoplaced)
+    (effects (font (size 1.27 1.27)) (justify left))
+    (property "Intersheetrefs" "${INTERSHEET_REFS}" (at 102.7036 72.39 0)
+      (effects (font (size 1.27 1.27)) (justify left) hide)
+    )
+  )
+  (global_label "L Line In" (shape input) (at 90.17 148.59 0) (fields_autoplaced)
+    (effects (font (size 1.27 1.27)) (justify left))
+    (property "Intersheetrefs" "${INTERSHEET_REFS}" (at 101.2522 148.59 0)
+      (effects (font (size 1.27 1.27)) (justify left) hide)
+    )
+  )
+  (symbol (lib_id "power:GND") (at 86.36 116.84 0) (unit 1)
+    (in_bom yes) (on_board yes) (dnp no) (fields_autoplaced)
+    (property "Reference" "#PWR013" (at 86.36 123.19 0)
+      (effects (font (size 1.27 1.27)) hide)
+    )
+    (property "Value" "GND" (at 86.36 121.92 0)
+      (effects (font (size 1.27 1.27)))
+    )
+    (property "Footprint" "" (at 86.36 116.84 0)
+      (effects (font (size 1.27 1.27)) hide)
+    )
+    (property "Datasheet" "" (at 86.36 116.84 0)
+      (effects (font (size 1.27 1.27)) hide)
+    )
+    (pin "1")
+    (instances
+      (project "teensy-dsp"
+        (path "/b4828465-e4d8-4e3f-b668-f3defd59a393/a9acb021-a9c9-4966-bb52-01ef79e2b2e6"
+          (reference "#PWR013") (unit 1)
+        )
+      )
+    )
   )
   (symbol (lib_id "2023-11-11_03-32-11:ACJS-IH") (at 81.28 64.77 0) (unit 1)
@@
     )
   )
+  (symbol (lib_id "power:GND") (at 86.36 40.64 0) (unit 1)
+    (in_bom yes) (on_board yes) (dnp no) (fields_autoplaced)
+    (property "Reference" "#PWR015" (at 86.36 46.99 0)
+      (effects (font (size 1.27 1.27)) hide)
+    )
+    (property "Value" "GND" (at 86.36 45.72 0)
+      (effects (font (size 1.27 1.27)))
+    )
+    (property "Footprint" "" (at 86.36 40.64 0)
+      (effects (font (size 1.27 1.27)) hide)
+    )
+    (property "Datasheet" "" (at 86.36 40.64 0)
+      (effects (font (size 1.27 1.27)) hide)
+    )
+    (pin "1")
+    (instances
+      (project "teensy-dsp"
+        (path "/b4828465-e4d8-4e3f-b668-f3defd59a393/a9acb021-a9c9-4966-bb52-01ef79e2b2e6"
+          (reference "#PWR015") (unit 1)
+        )
+      )
+    )
+  )
   (symbol (lib_id "2023-11-11_03-32-11:ACJS-IH") (at 81.28 115.57 0) (unit 1)
     (in_bom yes) (on_board yes) (dnp no) (fields_autoplaced)
@@
     )
   )
+  (symbol (lib_id "power:GND") (at 86.36 66.04 0) (unit 1)
+    (in_bom yes) (on_board yes) (dnp no) (fields_autoplaced)
+    (property "Reference" "#PWR014" (at 86.36 72.39 0)
+      (effects (font (size 1.27 1.27)) hide)
+    )
+    (property "Value" "GND" (at 86.36 71.12 0)
+      (effects (font (size 1.27 1.27)))
+    )
+    (property "Footprint" "" (at 86.36 66.04 0)
+      (effects (font (size 1.27 1.27)) hide)
+    )
+    (property "Datasheet" "" (at 86.36 66.04 0)
+      (effects (font (size 1.27 1.27)) hide)
+    )
+    (pin "1")
+    (instances
+      (project "teensy-dsp"
+        (path "/b4828465-e4d8-4e3f-b668-f3defd59a393/a9acb021-a9c9-4966-bb52-01ef79e2b2e6"
+          (reference "#PWR014") (unit 1)
+        )
+      )
+    )
+  )
   (symbol (lib_id "2023-11-11_03-32-11:ACJS-IH") (at 81.28 140.97 0) (unit 1)
     (in_bom yes) (on_board yes) (dnp no) (fields_autoplaced)
@@
         )
       )
+    )
+  )
+  (symbol (lib_id "power:GND") (at 86.36 142.24 0) (unit 1)
+    (in_bom yes) (on_board yes) (dnp no) (fields_autoplaced)
+    (property "Reference" "#PWR012" (at 86.36 148.59 0)
+      (effects (font (size 1.27 1.27)) hide)
+    )
+    (property "Value" "GND" (at 86.36 147.32 0)
+      (effects (font (size 1.27 1.27)))
+    )
+    (property "Footprint" "" (at 86.36 142.24 0)
+      (effects (font (size 1.27 1.27)) hide)
+    )
+    (property "Datasheet" "" (at 86.36 142.24 0)
+      (effects (font (size 1.27 1.27)) hide)
+    )
+    (pin "1")
+    (instances
+      (project "teensy-dsp"
+        (path "/b4828465-e4d8-4e3f-b668-f3defd59a393/a9acb021-a9c9-4966-bb52-01ef79e2b2e6"
+          (reference "#PWR012") (unit 1)
+        )
+      )

Commit message: update pcb layout
Connections:
- net L Line In: now also J1.T; no longer J2.T
- net L Line Out: now also J1.T; no longer J2.T
- net R Line In: now also J2.T; no longer J1.T
- net R Line Out: now also J2.T; no longer J1.T
Changed lines of the file:
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@@
     (stroke (width 0) (type default))
   )
-  (wire (pts (xy 81.28 46.99) (xy 90.17 46.99))
+  (wire (pts (xy 81.28 46.99) (xy 88.9 46.99))
+    (stroke (width 0) (type default))
+  )
+  (wire (pts (xy 81.28 123.19) (xy 88.9 123.19))
     (stroke (width 0) (type default))
   )
@@
     (stroke (width 0) (type default))
   )
-  (wire (pts (xy 81.28 72.39) (xy 90.17 72.39))
+  (wire (pts (xy 86.36 64.77) (xy 86.36 66.04))
     (stroke (width 0) (type default))
   )
-  (wire (pts (xy 86.36 64.77) (xy 86.36 66.04))
+  (wire (pts (xy 81.28 72.39) (xy 88.9 72.39))
     (stroke (width 0) (type default))
   )
@@
     (stroke (width 0) (type default))
   )
-  (wire (pts (xy 81.28 123.19) (xy 90.17 123.19))
+  (wire (pts (xy 81.28 148.59) (xy 88.9 148.59))
     (stroke (width 0) (type default))
   )
@@
     (stroke (width 0) (type default))
   )
-  (wire (pts (xy 81.28 148.59) (xy 90.17 148.59))
-    (stroke (width 0) (type default))
-  )
-  (text "Left Output" (at 60.96 81.28 0)
+  (text "Left Output" (at 60.96 132.08 0)
     (effects (font (size 1.27 1.27)) (justify left bottom))
   )
-  (text "Right Ouptut" (at 60.96 55.88 0)
+  (text "Right Ouptut" (at 60.96 157.48 0)
     (effects (font (size 1.27 1.27)) (justify left bottom))
   )
-  (text "Left Input" (at 60.96 157.48 0)
+  (text "Left Input" (at 60.96 55.88 0)
     (effects (font (size 1.27 1.27)) (justify left bottom))
   )
-  (text "Right Input" (at 60.96 132.08 0)
+  (text "Right Input" (at 60.96 81.28 0)
     (effects (font (size 1.27 1.27)) (justify left bottom))
   )
-  (global_label "R Line Out" (shape input) (at 90.17 46.99 0) (fields_autoplaced)
+  (global_label "R Line Out" (shape input) (at 88.9 148.59 0) (fields_autoplaced)
     (effects (font (size 1.27 1.27)) (justify left))
-    (property "Intersheetrefs" "${INTERSHEET_REFS}" (at 102.9455 46.99 0)
+    (property "Intersheetrefs" "${INTERSHEET_REFS}" (at 101.6755 148.59 0)
       (effects (font (size 1.27 1.27)) (justify left) hide)
     )
   )
-  (global_label "R Line In" (shape input) (at 90.17 123.19 0) (fields_autoplaced)
+  (global_label "R Line In" (shape input) (at 88.9 72.39 0) (fields_autoplaced)
     (effects (font (size 1.27 1.27)) (justify left))
-    (property "Intersheetrefs" "${INTERSHEET_REFS}" (at 101.4941 123.19 0)
+    (property "Intersheetrefs" "${INTERSHEET_REFS}" (at 100.2241 72.39 0)
       (effects (font (size 1.27 1.27)) (justify left) hide)
     )
   )
-  (global_label "L Line Out" (shape input) (at 90.17 72.39 0) (fields_autoplaced)
+  (global_label "L Line Out" (shape input) (at 88.9 123.19 0) (fields_autoplaced)
     (effects (font (size 1.27 1.27)) (justify left))
-    (property "Intersheetrefs" "${INTERSHEET_REFS}" (at 102.7036 72.39 0)
+    (property "Intersheetrefs" "${INTERSHEET_REFS}" (at 101.4336 123.19 0)
       (effects (font (size 1.27 1.27)) (justify left) hide)
     )
   )
-  (global_label "L Line In" (shape input) (at 90.17 148.59 0) (fields_autoplaced)
+  (global_label "L Line In" (shape input) (at 88.9 46.99 0) (fields_autoplaced)
     (effects (font (size 1.27 1.27)) (justify left))
-    (property "Intersheetrefs" "${INTERSHEET_REFS}" (at 101.2522 148.59 0)
+    (property "Intersheetrefs" "${INTERSHEET_REFS}" (at 99.9822 46.99 0)
       (effects (font (size 1.27 1.27)) (justify left) hide)
     )

Commit message: case updates
Parts:
- removed J2: ACJS-IH, ACJS-IH_AMP, symbol 2023-11-11_03-32-11:ACJS-IH
- added C4, C5: 1uF 50V, symbol Device:C
- added J1: ACJS-IH, ACJS-IH_AMP, symbol 2023-11-11_03-32-11:ACJS-IH
- added R2, R4: 1M, symbol Device:R
- added R3, R5: 1k, symbol Device:R
- added RV1, RV2: 10k, symbol Device:R_Potentiometer
- added SW1: SW_DPDT_x2, symbol Switch:SW_DPDT_x2
- added U4: TL074, symbol Amplifier_Operational:TL074
Connections:
- net GND: now also J1.R, R2.2, R4.2, RV1.1, RV2.1, U4.10 (+), U4.11 (V-), U4.12 (+), U4.13 (-), U4.9 (-)
- net L Line In: now also SW1.2 (B); no longer J1.T
- net R Line In: now also SW1.5 (B)
- new net: C5.1, R4.1
- new net: C5.2, U4.5 (+)
- new net: R3.1, RV1.2
- new net: RV1.3, SW1.1 (A), U4.1
- new net: J1.T, SW1.6 (C)
- new net: R5.2, U4.6 (-)
- new net: RV2.3, SW1.4 (A), U4.7
- new net: R3.2, U4.2 (-)
- new net: J1.T, SW1.3 (C)
- new net: C4.2, U4.3 (+)
- new net: R5.1, RV2.2
- new net: C4.1, R2.1
- new net +9V: U4.4 (V+)
- no-connect marks 16 -> 18
Other:
- moved on the sheet: J1, J2
