File: pcb/teensy-dsp/teensy-dsp-frontend/teensy-dsp-frontend.kicad_pcb (KiCad board)
At the start: 4 copper layers, 88 x 75 mm, 18 parts, among them J1 Conn_02x15_Odd_Even, U1 TLC5940PWP

Commit message: update renders
Routing:
- net POT_1: track 0.00 -> 57.1 mm
- net POT_5: track 0.00 -> 54.7 mm
- net POT_3: track 0.00 -> 41.7 mm
- net POT_6: track 0.14 -> 41.1 mm
- net POT_2: track 0.00 -> 31.3 mm
- net POT_4: track 1.47 -> 14.1 mm
- net Net-(U1-GSCLK): track 8.96 -> 0.00 mm
- added copper zone on In2.Cu, net +3.3V
- added copper zone on In2.Cu, net +9V
- added copper zone on In1.Cu, net GND
Changed lines of the file:
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@@
   (gr_arc (start 54 106) (mid 52.585786 105.414214) (end 52 104)
     (stroke (width 0.1) (type default)) (layer "Edge.Cuts"))
-  (segment (start 71.3 74.58) (end 80.26 74.58) (width 0.25) (layer "B.Cu") (net 13))
   (segment (start 136.723949 86.223949) (end 137.173949 86.673949) (width 0.25) (layer "B.Cu") (net 19))
   (segment (start 136.723949 81.143949) (end 136.723949 81.453949) (width 0.25) (layer "B.Cu") (net 21))
+  (segment (start 58.775 73.775) (end 67 82) (width 0.25) (layer "F.Cu") (net 23))
+  (segment (start 67 82) (end 80.88 82) (width 0.25) (layer "F.Cu") (net 23))
+  (segment (start 80.88 82) (end 83.023949 84.143949) (width 0.25) (layer "F.Cu") (net 23))
+  (segment (start 60 45.725) (end 58.775 46.95) (width 0.25) (layer "F.Cu") (net 23))
+  (segment (start 58.775 46.95) (end 58.775 73.775) (width 0.25) (layer "F.Cu") (net 23))
   (segment (start 96 72.725) (end 96.767588 72.725) (width 0.25) (layer "F.Cu") (net 25))
-  (segment (start 108.186537 84.143949) (end 108.883949 84.143949) (width 0.25) (layer "F.Cu") (net 25))
+  (segment (start 96 79) (end 91 84) (width 0.25) (layer "F.Cu") (net 25))
+  (segment (start 96 72.725) (end 96 79) (width 0.25) (layer "F.Cu") (net 25))
+  (segment (start 61.225 71.5) (end 72.92 71.5) (width 0.25) (layer "F.Cu") (net 26))
+  (segment (start 60 72.725) (end 61.225 71.5) (width 0.25) (layer "F.Cu") (net 26))
+  (segment (start 72.92 71.5) (end 85.563949 84.143949) (width 0.25) (layer "F.Cu") (net 26))
+  (segment (start 93.581051 84.143949) (end 93.183949 84.143949) (width 0.25) (layer "F.Cu") (net 27))
+  (segment (start 132 45.725) (end 93.581051 84.143949) (width 0.25) (layer "F.Cu") (net 27))
+  (segment (start 96 45.725) (end 88.103949 53.621051) (width 0.25) (layer "F.Cu") (net 28))
+  (segment (start 88.103949 53.621051) (end 88.103949 84.143949) (width 0.25) (layer "F.Cu") (net 28))
   (segment (start 132 72.725) (end 132 72.867898) (width 0.25) (layer "F.Cu") (net 29))
+  (segment (start 130.775 73.95) (end 105.917898 73.95) (width 0.25) (layer "F.Cu") (net 29))
+  (segment (start 132 72.725) (end 130.775 73.95) (width 0.25) (layer "F.Cu") (net 29))
+  (segment (start 105.917898 73.95) (end 95.723949 84.143949) (width 0.25) (layer "F.Cu") (net 29))
+  (zone (net 11) (net_name "GND") (layer "In1.Cu") (hatch edge 0.5)
+    (connect_pads (clearance 0.5))
+    (min_thickness 0.25) (filled_areas_thickness no)
+    (fill yes (thermal_gap 0.5) (thermal_bridge_width 0.5))
+    (polygon
+      (pts
+        (xy 52 31)
+        (xy 140 31)
+        (xy 140 106)
+        (xy 52 106)
+      )
+    )
+  )
+  (zone (net 24) (net_name "+3.3V") (layer "In2.Cu") (hatch edge 0.5)
+    (priority 1)
+    (connect_pads (clearance 0.5))
+    (min_thickness 0.25) (filled_areas_thickness no)
+    (fill yes (thermal_gap 0.5) (thermal_bridge_width 0.5))
+    (polygon
+      (pts
+        (xy 52 31)
+        (xy 140 31)
+        (xy 140 95)
+        (xy 67 95)
+        (xy 67 81)
+        (xy 52 81)
+      )
+    )
+  )
+  (zone (net 2) (net_name "+9V") (layer "In2.Cu") (hatch edge 0.5)
+    (priority 2)
+    (connect_pads (clearance 0.5))
+    (min_thickness 0.25) (filled_areas_thickness no)
+    (fill yes (thermal_gap 0.5) (thermal_bridge_width 0.5))
+    (polygon
+      (pts
+        (xy 52 81)
+        (xy 67 81)
+        (xy 67 95)
+        (xy 140 95)
+        (xy 140 106)
+        (xy 52 106)
+      )
+    )
+  )
 )

Commit message: pcb and case updates
Parts:
- removed D1, D2, D3: LED_RABG, LED_THT:LED_D5.0mm-4_RGB_Staggered_Pins
- added J2: Conn_01x04_Pin, Connector_PinHeader_2.54mm:PinHeader_1x04_P2.54mm_Horizontal, B.Cu at (166.7, 112.6)
- added J3: Conn_01x04_Pin, Connector_PinHeader_2.54mm:PinHeader_1x04_P2.54mm_Horizontal, B.Cu at (154.7, 112.6)
- added J4: Conn_01x04_Pin, Connector_PinHeader_2.54mm:PinHeader_1x04_P2.54mm_Horizontal, B.Cu at (130.7, 112.6)
- added R7: 10k, Resistor_SMD:R_1206_3216Metric_Pad1.30x1.75mm_HandSolder, B.Cu at (168.4, 93.0)
- moved J1 86.5 mm to (144.8, 102.0), turned to 90 degrees
- moved RV1 69.0 mm to (108.0, 92.7)
- moved RV2 69.0 mm to (108.0, 119.7)
- moved RV4 69.0 mm to (143.9, 119.7)
- moved RV6 69.0 mm to (179.9, 119.7)
- moved RV3 69.0 mm to (143.9, 92.7)
- moved RV5 69.0 mm to (179.9, 92.7)
- moved R3 55.3 mm to (168.4, 90.0)
- moved C1 51.5 mm to (161.4, 97.0), turned to 0 degrees
- moved R1 51.1 mm to (161.4, 100.0)
- moved R2 50.8 mm to (161.4, 103.0)
- moved R6 49.8 mm to (179.4, 104.0), turned to 0 degrees
- moved U1 49.3 mm to (170.1, 101.0)
- moved R5 46.7 mm to (179.4, 101.0), turned to 0 degrees
- moved R4 44.8 mm to (179.4, 98.0), turned to 0 degrees
Routing:
- net +3.3V: track 0.00 -> 230.6 mm, vias 0 -> 1
- net LED_SIN: track 0.00 -> 76.5 mm
- net LED_SCLK: track 0.00 -> 69.4 mm
- net POT_5: track 54.7 -> 117.1 mm
- net LED_XLAT: track 0.00 -> 61.6 mm
- net POT_6: track 41.1 -> 97.0 mm
- net +9V: track 0.00 -> 55.7 mm
- net Net-(J4-Pin_2): track 0.00 -> 42.8 mm
- net Net-(J4-Pin_4): track 0.00 -> 41.0 mm
- net POT_1: track 57.1 -> 16.5 mm
- net Net-(J4-Pin_1): track 0.00 -> 39.6 mm
- net LED_BLANK: track 0.00 -> 39.4 mm
- net POT_4: track 14.1 -> 40.5 mm
- net LED_GSCLK: track 0.00 -> 25.8 mm
- net Net-(J3-Pin_1): track 0.00 -> 25.5 mm
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- added copper zone on B.Cu, net GND
- added copper zone on F.Cu, net GND
- removed copper zone on In2.Cu, net +3.3V
- removed copper zone on In2.Cu, net +9V
- removed copper zone on In1.Cu, net GND
Other:
- board size 88 x 75 mm -> 88 x 45 mm
- copper layers 4 -> 2
