File: pcb/teensy-dsp/teensy-dsp-frontend/teensy-dsp-frontend.kicad_sch (KiCad schematic)
At the start: 16 parts, among them U1 TLC5940PWP

Commit message: update renders
Parts:
- added C1: 100n, Capacitor_SMD:C_1206_3216Metric_Pad1.33x1.80mm_HandSolder, symbol Device:C
- added J1: Conn_02x15_Odd_Even, Connector_IDC:IDC-Header_2x15_P2.54mm_Vertical, symbol Connector_Generic:Conn_02x15_Odd_Even
- RV1, RV2, RV3, RV4, RV5, RV6: footprint Potentiometer_THT:Potentiometer_TT_P0915N -> Custom Potentiometers:Potentiometer_TT_P0915N
Connections:
- net +3.3V: now also C1.2, J1.7 (Pin_7)
- net +9V: now also J1.1 (Pin_1), J1.3 (Pin_3)
- net GND: now also C1.1, J1.10 (Pin_10), J1.12 (Pin_12), J1.14 (Pin_14), J1.16 (Pin_16), J1.18 (Pin_18), J1.2 (Pin_2), J1.20 (Pin_20), J1.22 (Pin_22), J1.24 (Pin_24), J1.26 (Pin_26), J1.28 (Pin_28), J1.30 (Pin_30), J1.4 (Pin_4), J1.6 (Pin_6), J1.8 (Pin_8)
- net LED_BLANK: now also J1.11 (Pin_11)
- net LED_GSCLK: now also J1.9 (Pin_9)
- net LED_SCLK: now also J1.15 (Pin_15)
- net LED_SIN: now also J1.17 (Pin_17)
- net LED_XLAT: now also J1.13 (Pin_13)
- net POT_1: now also J1.19 (Pin_19)
- net POT_2: now also RV2.2, J1.21 (Pin_21); no longer RV3.2
- net POT_3: now also RV3.2, J1.23 (Pin_23); no longer RV5.2
- net POT_4: now also RV4.2, J1.25 (Pin_25); no longer RV2.2
- net POT_5: now also RV5.2, J1.27 (Pin_27); no longer RV4.2
- net POT_6: now also J1.29 (Pin_29)
- new net +5V: J1.5 (Pin_5)
Other:
- moved on the sheet: D1, D2, D3, R1, R2, R3, R4, R5, R6, RV1, RV2, RV3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

Commit message: update pcb layout
Parts:
- added R7: 10k, Resistor_SMD:R_1206_3216Metric_Pad1.30x1.75mm_HandSolder, symbol Device:R
Connections:
- net +3.3V: now also R7.2
- net at R3.1, U1.2 (BLANK): now also R7.1
Other:
- moved on the sheet: J1, R3, R4, R5, R6

Commit message: pcb and case updates
Parts:
- removed D1, D2, D3: LED_RABG, LED_THT:LED_D5.0mm-4_RGB_Staggered_Pins, symbol Device:LED_RABG
- added J2, J3, J4: Conn_01x04_Pin, Connector_PinHeader_2.54mm:PinHeader_1x04_P2.54mm_Horizontal, symbol Connector:Conn_01x04_Pin
Connections:
- net +9V: now also J2.3 (Pin_3), J3.3 (Pin_3), J4.3 (Pin_3)
- net at U1.7 (OUT0): now also J2.4 (Pin_4)
- net at U1.9 (OUT2): now also J2.1 (Pin_1)
- net at U1.8 (OUT1): now also J2.2 (Pin_2)
- net at U1.13 (OUT6): now also J4.4 (Pin_4)
- net at U1.15 (OUT8): now also J4.1 (Pin_1)
- net at U1.14 (OUT7): now also J4.2 (Pin_2)
- net at U1.10 (OUT3): now also J3.4 (Pin_4)
- net at U1.11 (OUT4): now also J3.2 (Pin_2)
- net at U1.12 (OUT5): now also J3.1 (Pin_1)
